File: hardware/data_logger_esp32c3/data_logger_esp32c3.kicad_sch (KiCad schematic)
At the start: 72 parts, among them U1 ESP32-C3-MINI-1, U10 A03401A, U11 SX1509BIULTRT, U2 AZ1117IH-3.3TRG1, U4 LM321MF, U5 LM321MF, U6 LM321MF, U7 LM321MF, U8 LM321MF, U9 A03401A

Commit message: more layout
Parts:
- renumbered I2C_SCL1 to SCL1, I2C_SDA1 to SDA1
Other:
- moved on the sheet: SCL1, SDA1
Changed lines of the file:
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@@
     (stroke (width 0) (type default) (color 0 0 0 0))
   )
-  (wire (pts (xy 144.78 155.575) (xy 158.115 155.575))
+  (wire (pts (xy 144.78 155.575) (xy 156.21 155.575))
     (stroke (width 0) (type default) (color 0 0 0 0))
   )
@@
     (stroke (width 0) (type default) (color 0 0 0 0))
   )
-  (wire (pts (xy 147.955 153.035) (xy 156.21 153.035))
+  (wire (pts (xy 147.955 153.035) (xy 154.305 153.035))
     (stroke (width 0) (type default) (color 0 0 0 0))
   )
@@
     (pin "1")
   )
-  (symbol (lib_id "Connector:TestPoint") (at 158.115 155.575 0) (unit 1)
-    (in_bom yes) (on_board yes)
-    (property "Reference" "I2C_SCL1" (id 0) (at 159.385 154.305 0)
-      (effects (font (size 1.27 1.27)) (justify left))
-    )
-    (property "Value" "TestPoint" (id 1) (at 160.655 153.5429 0)
-      (effects (font (size 1.27 1.27)) (justify left) hide)
-    )
-    (property "Footprint" "TestPoint:TestPoint_THTPad_1.0x1.0mm_Drill0.5mm" (id 2) (at 163.195 155.575 0)
-      (effects (font (size 1.27 1.27)) hide)
-    )
-    (property "Datasheet" "~" (id 3) (at 163.195 155.575 0)
+  (symbol (lib_id "Connector:TestPoint") (at 156.21 155.575 0) (unit 1)
+    (in_bom yes) (on_board yes)
+    (property "Reference" "SCL1" (id 0) (at 157.48 154.305 0)
+      (effects (font (size 1.27 1.27)) (justify left))
+    )
+    (property "Value" "TestPoint" (id 1) (at 158.75 153.5429 0)
+      (effects (font (size 1.27 1.27)) (justify left) hide)
+    )
+    (property "Footprint" "TestPoint:TestPoint_THTPad_1.0x1.0mm_Drill0.5mm" (id 2) (at 161.29 155.575 0)
+      (effects (font (size 1.27 1.27)) hide)
+    )
+    (property "Datasheet" "~" (id 3) (at 161.29 155.575 0)
       (effects (font (size 1.27 1.27)) hide)
     )
@@
     (pin "2")
   )
-  (symbol (lib_id "Connector:TestPoint") (at 156.21 153.035 0) (unit 1)
-    (in_bom yes) (on_board yes)
-    (property "Reference" "I2C_SDA1" (id 0) (at 158.75 149.86 0)
-      (effects (font (size 1.27 1.27)) (justify left))
-    )
-    (property "Value" "TestPoint" (id 1) (at 158.75 151.0029 0)
-      (effects (font (size 1.27 1.27)) (justify left) hide)
-    )
-    (property "Footprint" "TestPoint:TestPoint_THTPad_1.0x1.0mm_Drill0.5mm" (id 2) (at 161.29 153.035 0)
-      (effects (font (size 1.27 1.27)) hide)
-    )
-    (property "Datasheet" "~" (id 3) (at 161.29 153.035 0)
+  (symbol (lib_id "Connector:TestPoint") (at 154.305 153.035 0) (unit 1)
+    (in_bom yes) (on_board yes)
+    (property "Reference" "SDA1" (id 0) (at 156.845 149.86 0)
+      (effects (font (size 1.27 1.27)) (justify left))
+    )
+    (property "Value" "TestPoint" (id 1) (at 156.845 151.0029 0)
+      (effects (font (size 1.27 1.27)) (justify left) hide)
+    )
+    (property "Footprint" "TestPoint:TestPoint_THTPad_1.0x1.0mm_Drill0.5mm" (id 2) (at 159.385 153.035 0)
+      (effects (font (size 1.27 1.27)) hide)
+    )
+    (property "Datasheet" "~" (id 3) (at 159.385 153.035 0)
       (effects (font (size 1.27 1.27)) hide)
     )
@@
       (reference "DC-1") (unit 1) (value "TestPoint") (footprint "TestPoint:TestPoint_THTPad_1.0x1.0mm_Drill0.5mm")
     )
-    (path "/17dbdba8-b282-4464-bba1-6a020e0bf650"
-      (reference "I2C_SCL1") (unit 1) (value "TestPoint") (footprint "TestPoint:TestPoint_THTPad_1.0x1.0mm_Drill0.5mm")
-    )
-    (path "/67ce0672-6e4f-43e5-9bb8-871700c947f7"
-      (reference "I2C_SDA1") (unit 1) (value "TestPoint") (footprint "TestPoint:TestPoint_THTPad_1.0x1.0mm_Drill0.5mm")
-    )
     (path "/6a8cc1dc-cdfe-4400-9f01-9b4ff95f0039"
       (reference "I2SN1") (unit 1) (value "TestPoint") (footprint "TestPoint:TestPoint_THTPad_1.0x1.0mm_Drill0.5mm")
@@
       (reference "RX0") (unit 1) (value "TestPoint") (footprint "TestPoint:TestPoint_THTPad_1.0x1.0mm_Drill0.5mm")
     )
+    (path "/17dbdba8-b282-4464-bba1-6a020e0bf650"
+      (reference "SCL1") (unit 1) (value "TestPoint") (footprint "TestPoint:TestPoint_THTPad_1.0x1.0mm_Drill0.5mm")
+    )
     (path "/a17f40b7-49cc-460a-8213-3c4690d2d239"
       (reference "SD1") (unit 1) (value "472192001") (footprint "1_project_footprints:472192001")
     )
+    (path "/67ce0672-6e4f-43e5-9bb8-871700c947f7"
+      (reference "SDA1") (unit 1) (value "TestPoint") (footprint "TestPoint:TestPoint_THTPad_1.0x1.0mm_Drill0.5mm")
+    )
     (path "/de8b7a30-7f1e-42b1-b9b4-5dde725e18cf"

Commit message: commit before routing
Parts:
- added R? (x2): 30.1, Resistor_SMD:R_0402_1005Metric, symbol Device:R_Small
Connections:
- net D+: now also R?.1; no longer USB-C1.A6 (DP1), USB-C1.B6 (DP2)
- net D-: now also R?.1; no longer USB-C1.A7 (DN1), USB-C1.B7 (DN2)
- new net: R?.2, USB-C1.A6 (DP1), USB-C1.B6 (DP2)
- new net: R?.2, USB-C1.A7 (DN1), USB-C1.B7 (DN2)
