File: hardware/data_logger_esp32c3/data_logger_esp32c3.kicad_sch (KiCad schematic)
At the start: 74 parts, among them U1 ESP32-C3-MINI-1, U10 A03401A, U11 SX1509BIULTRT, U2 AZ1117IH-3.3TRG1, U4 LM321MF, U5 LM321MF, U6 LM321MF, U7 LM321MF, U8 LM321MF, U9 A03401A

Commit message: routing done
Parts:
- gave numbers to parts that had none: 2
Connections:
- net D_CONN+: now reaches R17.2, USB-C1.A6 (DP1), USB-C1.B6 (DP2)
- net D_CONN-: now reaches R18.2, USB-C1.A7 (DN1), USB-C1.B7 (DN2)
Other:
- moved on the sheet: R17, R18
Changed lines of the file:
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@@
     (stroke (width 0) (type default) (color 0 0 0 0))
   )
-  (wire (pts (xy 181.61 62.23) (xy 183.515 62.23))
+  (wire (pts (xy 181.61 62.23) (xy 193.675 62.23))
     (stroke (width 0) (type default) (color 0 0 0 0))
   )
@@
     (stroke (width 0) (type default) (color 0 0 0 0))
   )
-  (wire (pts (xy 181.61 55.88) (xy 183.515 55.88))
+  (wire (pts (xy 181.61 55.88) (xy 193.675 55.88))
     (stroke (width 0) (type default) (color 0 0 0 0))
   )
@@
     )
   )
-  (global_label "D+" (shape input) (at 188.595 55.88 0) (fields_autoplaced)
+  (global_label "D+" (shape input) (at 198.755 55.88 0) (fields_autoplaced)
     (effects (font (size 1.27 1.27)) (justify left))
-    (property "Intersheet References" "${INTERSHEET_REFS}" (id 0) (at 193.8505 55.8006 0)
+    (property "Intersheet References" "${INTERSHEET_REFS}" (id 0) (at 204.0105 55.8006 0)
       (effects (font (size 1.27 1.27)) (justify left) hide)
     )
@@
     )
   )
-  (global_label "D-" (shape input) (at 188.595 62.23 0) (fields_autoplaced)
+  (global_label "D-" (shape input) (at 198.755 62.23 0) (fields_autoplaced)
     (effects (font (size 1.27 1.27)) (justify left))
-    (property "Intersheet References" "${INTERSHEET_REFS}" (id 0) (at 193.8505 62.1506 0)
+    (property "Intersheet References" "${INTERSHEET_REFS}" (id 0) (at 204.0105 62.1506 0)
+      (effects (font (size 1.27 1.27)) (justify left) hide)
+    )
+  )
+  (global_label "D_CONN+" (shape input) (at 187.325 55.88 90) (fields_autoplaced)
+    (effects (font (size 1.27 1.27)) (justify left))
+    (property "Intersheet References" "${INTERSHEET_REFS}" (id 0) (at 187.2456 44.3955 90)
       (effects (font (size 1.27 1.27)) (justify left) hide)
     )
@@
     (effects (font (size 1.27 1.27)) (justify right))
     (property "Intersheet References" "${INTERSHEET_REFS}" (id 0) (at 42.0974 180.2606 0)
+      (effects (font (size 1.27 1.27)) (justify right) hide)
+    )
+  )
+  (global_label "D_CONN-" (shape input) (at 187.325 62.23 270) (fields_autoplaced)
+    (effects (font (size 1.27 1.27)) (justify right))
+    (property "Intersheet References" "${INTERSHEET_REFS}" (id 0) (at 187.2456 73.7145 90)
       (effects (font (size 1.27 1.27)) (justify right) hide)
     )
@@
     (pin "1")
   )
-  (symbol (lib_id "Device:R_Small") (at 186.055 62.23 270) (unit 1)
-    (in_bom yes) (on_board yes)
-    (property "Reference" "R?" (id 0) (at 187.325 58.42 90)
+  (symbol (lib_id "Device:R_Small") (at 196.215 62.23 270) (unit 1)
+    (in_bom yes) (on_board yes)
+    (property "Reference" "R18" (id 0) (at 197.485 58.42 90)
       (effects (font (size 1.27 1.27)) (justify right))
     )
-    (property "Value" "30.1" (id 1) (at 188.595 60.325 90)
+    (property "Value" "30.1" (id 1) (at 198.755 60.325 90)
       (effects (font (size 1.27 1.27)) (justify right))
     )
-    (property "Footprint" "Resistor_SMD:R_0402_1005Metric" (id 2) (at 186.055 62.23 0)
-      (effects (font (size 1.27 1.27)) hide)
-    )
-    (property "Datasheet" "~" (id 3) (at 186.055 62.23 0)
-      (effects (font (size 1.27 1.27)) hide)
-    )
-    (property "part_number" "0402WGF301JTCE" (id 4) (at 186.055 62.23 0)
+    (property "Footprint" "Resistor_SMD:R_0402_1005Metric" (id 2) (at 196.215 62.23 0)
+      (effects (font (size 1.27 1.27)) hide)
+    )
+    (property "Datasheet" "~" (id 3) (at 196.215 62.23 0)
+      (effects (font (size 1.27 1.27)) hide)
+    )
+    (property "part_number" "0402WGF301JTCE" (id 4) (at 196.215 62.23 0)
       (effects (font (size 1.27 1.27)) hide)
     )
@@
     (pin "1")
   )
-  (symbol (lib_id "Device:R_Small") (at 186.055 55.88 270) (unit 1)
-    (in_bom yes) (on_board yes)
-    (property "Reference" "R?" (id 0) (at 187.325 52.07 90)
+  (symbol (lib_id "Device:R_Small") (at 196.215 55.88 270) (unit 1)
+    (in_bom yes) (on_board yes)
+    (property "Reference" "R17" (id 0) (at 197.485 52.07 90)
       (effects (font (size 1.27 1.27)) (justify right))
     )
-    (property "Value" "30.1" (id 1) (at 188.595 53.975 90)
+    (property "Value" "30.1" (id 1) (at 198.755 53.975 90)
       (effects (font (size 1.27 1.27)) (justify right))
     )
-    (property "Footprint" "Resistor_SMD:R_0402_1005Metric" (id 2) (at 186.055 55.88 0)
-      (effects (font (size 1.27 1.27)) hide)
-    )
-    (property "Datasheet" "~" (id 3) (at 186.055 55.88 0)
-      (effects (font (size 1.27 1.27)) hide)
-    )
-    (property "part_number" "0402WGF301JTCE" (id 4) (at 186.055 55.88 0)
+    (property "Footprint" "Resistor_SMD:R_0402_1005Metric" (id 2) (at 196.215 55.88 0)
+      (effects (font (size 1.27 1.27)) hide)
+    )
+    (property "Datasheet" "~" (id 3) (at 196.215 55.88 0)
+      (effects (font (size 1.27 1.27)) hide)
+    )
+    (property "part_number" "0402WGF301JTCE" (id 4) (at 196.215 55.88 0)
       (effects (font (size 1.27 1.27)) hide)
     )
@@
       (reference "R16") (unit 1) (value "4.7k") (footprint "Resistor_SMD:R_0402_1005Metric")
     )
+    (path "/7862a053-75e1-4422-9330-83a5aacef5b4"
+      (reference "R17") (unit 1) (value "30.1") (footprint "Resistor_SMD:R_0402_1005Metric")
+    )
     (path "/74f836ea-3bdb-4f8c-8310-211294f774e1"
-      (reference "R?") (unit 1) (value "30.1") (footprint "Resistor_SMD:R_0402_1005Metric")
-    )
-    (path "/7862a053-75e1-4422-9330-83a5aacef5b4"
-      (reference "R?") (unit 1) (value "30.1") (footprint "Resistor_SMD:R_0402_1005Metric")
+      (reference "R18") (unit 1) (value "30.1") (footprint "Resistor_SMD:R_0402_1005Metric")
     )
     (path "/be7b7f09-e1f8-49ba-84ba-cb32817ab458"

Commit message: more layout
Connections:
- net I2C_SCL: now also U1.13 (GPIO1/ADC1_CH1/XTAL_32K_N); no longer U1.16 (GPIO10)
- net I2C_SDA: now also U1.16 (GPIO10); no longer U1.13 (GPIO1/ADC1_CH1/XTAL_32K_N)
Changed lines of the file:
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@@
+    )
+  )
+  (global_label "I2C_SDA" (shape input) (at 55.245 61.595 180) (fields_autoplaced)
+    (effects (font (size 1.27 1.27)) (justify right))
+    (property "Intersheet References" "${INTERSHEET_REFS}" (id 0) (at 45.2119 61.5156 0)
+      (effects (font (size 1.27 1.27)) (justify right) hide)
     )
   )
@@
     )
   )
-  (global_label "I2C_SCL" (shape input) (at 55.245 61.595 180) (fields_autoplaced)
-    (effects (font (size 1.27 1.27)) (justify right))
-    (property "Intersheet References" "${INTERSHEET_REFS}" (id 0) (at 45.2724 61.5156 0)
-      (effects (font (size 1.27 1.27)) (justify right) hide)
-    )
-  )
   (global_label "SCLK" (shape input) (at 46.99 185.42 180) (fields_autoplaced)
     (effects (font (size 1.27 1.27)) (justify right))
@@
     (effects (font (size 1.27 1.27)) (justify right))
     (property "Intersheet References" "${INTERSHEET_REFS}" (id 0) (at 130.3019 152.9556 0)
+      (effects (font (size 1.27 1.27)) (justify right) hide)
+    )
+  )
+  (global_label "I2C_SCL" (shape input) (at 55.245 59.055 180) (fields_autoplaced)
+    (effects (font (size 1.27 1.27)) (justify right))
+    (property "Intersheet References" "${INTERSHEET_REFS}" (id 0) (at 45.2724 58.9756 0)
       (effects (font (size 1.27 1.27)) (justify right) hide)
     )
@@
       (effects (font (size 1.27 1.27)) (justify right) hide)
     )
-  )
-  (global_label "I2C_SDA" (shape input) (at 55.245 59.055 180) (fields_autoplaced)
-    (effects (font (size 1.27 1.27)) (justify right))
-    (property "Intersheet References" "${INTERSHEET_REFS}" (id 0) (at 45.2119 58.9756 0)
-      (effects (font (size 1.27 1.27)) (justify right) hide)
-    )
