File: hardware/data_logger_esp32c3/data_logger_esp32c3.kicad_pcb (KiCad board)
At the start: 4 copper layers, 43.3 x 32.3 mm, 74 parts, among them U1 ESP32-C3-MINI-1, U10 A03401A, U11 SX1509BIULTRT, U2 AZ1117IH-3.3TRG1, U4 LM321MF, U5 LM321MF, U6 LM321MF, U7 LM321MF, U8 LM321MF, U9 A03401A

Commit message: last commit for the night
Routing:
- net I2C_SCL: track 4.90 -> 27.4 mm, vias 0 -> 1
- net Net-(IO2-Pad1): track 0.00 -> 22.3 mm
- net Net-(IO0-Pad1): track 0.00 -> 21.7 mm
- net Net-(IO1-Pad1): track 0.00 -> 21.0 mm
- net I2C_SDA: track 6.19 -> 25.5 mm, vias 0 -> 1
- net Net-(IO8-Pad1): track 0.00 -> 14.7 mm
- net Net-(IO12-Pad1): track 0.00 -> 14.1 mm
- net Net-(IO15-Pad1): track 0.00 -> 13.6 mm
- net Net-(IO13-Pad1): track 0.00 -> 13.1 mm
- net GND: track 10.7 -> 23.8 mm, vias 18 -> 20
- net Net-(IO9-Pad1): track 0.00 -> 13.0 mm
- net Net-(IO3-Pad1): track 0.00 -> 12.8 mm, vias 0 -> 1
- net Net-(IO14-Pad1): track 0.00 -> 12.8 mm
- net NRESET: track 1.79 -> 14.3 mm, vias 0 -> 1
- net Net-(IO10-Pad1): track 0.00 -> 12.1 mm
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